File: Core/Pandoras box.kicad_pcb (KiCad board)
At the start: 4 copper layers, 80 x 43 mm, 120 parts, among them J1 JST_PH_S4B-PH-K, J2 JST_PH_S4B-PH-K, J3 JST_PH_S3B-PH-K, J4 JST_PH_S6B-PH-K, J5 JST_PH_S6B-PH-K, J6 Conn_02x06_Odd_Even, J7 Conn_01x02_Male, J8 Conn_01x02_Male, J9 Conn_02x06_Odd_Even, Q1 STD2805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

Commit message: Add partial routing
Parts:
- J7, J8: footprint Connector_PinSocket_2.54mm:PinSocket_1x02_P2.54mm_Vertical -> Connector_PinHeader_2.54mm:PinHeader_1x02_P2.54mm_Vertical
- moved J3 99.9 mm to (104.1, 83.8), turned to 180 degrees
- moved U2 42.0 mm to (161.3, 116.8), turned to 0 degrees
- moved D1 38.2 mm to (161.5, 73.9)
- moved R25 38.2 mm to (163.0, 74.4)
- moved J7 27.2 mm to (204.5, 87.6)
